File: hardware/rtc.sch (KiCad schematic (older format))
At the start: 11 parts, among them P1 CON-SENSOR, U1 M24C64, U4 DRILL, U5 DRILL, U6 DRILL, U7 DRILL

Commit message: fully routed
Parts:
- removed X?: CRYSTAL, symbol CRYSTAL
- added BT1: BATTERY, kicad-libraries:BATTERY_HOLDER_2998, symbol BATTERY
- added C3: 100nF, kicad-libraries:0603E, symbol C
- added X1: 32.768kHz, kicad-libraries:AB26TRQ, symbol CRYSTAL_3225
- RP1: renamed from RP?; value R_PACK4 -> 2k2; footprint 4X0603 -> kicad-libraries:4X0603
- U2: renamed from U?; footprint (none) -> kicad-libraries:SO-8
- gave numbers to parts that had none: 1
- renumbered C7 to C2, U4 to U3, U5 to U4, U6 to U5, U7 to U6
Connections:
- wire segments 43 -> 50
- no-connect marks 3 -> 4
Other:
- note added: "AB26TRQ-32.768kHz-T"
- note added: "CL = 6,7,12.5pF"
- note added: "Digikey 36-2998-ND"
Changed lines of the file:
@@
 LIBS:ac-dc
 LIBS:74xgxx
+LIBS:rtc-cache
 EELAYER 25 0
 EELAYER END
@@
 NoConn ~ 4250 2600
 $Comp
-L DRILL U4
+L DRILL U3
 U 1 1 4C6050A5
 P 10650 6150
-F 0 "U4" H 10700 6200 60  0001 C CNN
+F 0 "U3" H 10700 6200 60  0001 C CNN
 F 1 "DRILL" H 10650 6150 60  0000 C CNN
 F 2 "kicad-libraries:DRILL_NP" H 10650 6150 60  0001 C CNN
@@
 $EndComp
 $Comp
-L DRILL U5
+L DRILL U4
 U 1 1 4C6050A2
 P 10650 6350
-F 0 "U5" H 10700 6400 60  0001 C CNN
+F 0 "U4" H 10700 6400 60  0001 C CNN
 F 1 "DRILL" H 10650 6350 60  0000 C CNN
 F 2 "kicad-libraries:DRILL_NP" H 10650 6350 60  0001 C CNN
@@
 $EndComp
 $Comp
-L DRILL U7
+L DRILL U6
 U 1 1 4C60509F
 P 11000 6350
-F 0 "U7" H 11050 6400 60  0001 C CNN
+F 0 "U6" H 11050 6400 60  0001 C CNN
 F 1 "DRILL" H 11000 6350 60  0000 C CNN
 F 2 "kicad-libraries:DRILL_NP" H 11000 6350 60  0001 C CNN
@@
 $EndComp
 $Comp
-L DRILL U6
+L DRILL U5
 U 1 1 4C605099
 P 11000 6150
-F 0 "U6" H 11050 6200 60  0001 C CNN
+F 0 "U5" H 11050 6200 60  0001 C CNN
 F 1 "DRILL" H 11000 6150 60  0000 C CNN
 F 2 "kicad-libraries:DRILL_NP" H 11000 6150 60  0001 C CNN
@@
 $EndComp
 $Comp
-L C C7
+L C C2
 U 1 1 4C5FD6ED
 P 4500 2400
-F 0 "C7" V 4650 2400 50  0000 L CNN
+F 0 "C2" V 4650 2400 50  0000 L CNN
 F 1 "100nF" V 4350 2400 50  0000 L CNN
 F 2 "kicad-libraries:0603E" H 4500 2400 60  0001 C CNN
@@
 $EndComp
 $Comp
-L GND #PWR04
+L GND #PWR03
 U 1 1 4C5FCF5E
 P 2000 2250
-F 0 "#PWR04" H 2000 2250 30  0001 C CNN
+F 0 "#PWR03" H 2000 2250 30  0001 C CNN
 F 1 "GND" H 2000 2180 30  0001 C CNN
 F 2 "" H 2000 2250 60  0001 C CNN
@@
 $EndComp
 $Comp
-L GND #PWR05
+L GND #PWR04
 U 1 1 4C5FCF4F
 P 1400 3300
-F 0 "#PWR05" H 1400 3300 30  0001 C CNN
+F 0 "#PWR04" H 1400 3300 30  0001 C CNN
 F 1 "GND" H 1400 3230 30  0001 C CNN
 F 2 "" H 1400 3300 60  0001 C CNN
@@
 	2800 2700 2800 2650
 $Comp
-L 3V3 #PWR026
+L 3V3 #PWR05
 U 1 1 56434DEF
 P 4250 2400
-F 0 "#PWR026" H 4250 2500 40  0001 C CNN
+F 0 "#PWR05" H 4250 2500 40  0001 C CNN
 F 1 "3V3" H 4250 2525 40  0000 C CNN
 F 2 "" H 4250 2400 60  0000 C CNN
@@
 $EndComp
 $Comp
-L PCF85263AT U?
+L PCF85263AT U2
 U 1 1 56437698
 P 3900 4300
-F 0 "U?" H 4050 4550 60  0000 C CNN
+F 0 "U2" H 4050 4550 60  0000 C CNN
 F 1 "PCF85263AT" H 3900 4050 60  0000 C CNN
-F 2 "" H 4400 4100 60  0000 C CNN
+F 2 "kicad-libraries:SO-8" H 4400 4100 60  0001 C CNN
 F 3 "" H 4400 4100 60  0000 C CNN
 	1    3900 4300
@@
 $EndComp
 $Comp
-L C C?
+L C C1
 U 1 1 56437B41
 P 3900 3950
-F 0 "C?" V 4050 3950 50  0000 L CNN
+F 0 "C1" V 4050 3950 50  0000 L CNN
 F 1 "100nF" V 3850 3650 50  0000 L CNN
 F 2 "kicad-libraries:0603E" H 3900 3950 60  0001 C CNN
@@
 $EndComp
 $Comp
-L 3V3 #PWR?
+L 3V3 #PWR06
 U 1 1 56437C5A
 P 3500 3900
-F 0 "#PWR?" H 3500 4000 40  0001 C CNN
+F 0 "#PWR06" H 3500 4000 40  0001 C CNN
 F 1 "3V3" H 3500 4025 40  0000 C CNN
 F 2 "" H 3500 3900 60  0000 C CNN
@@
 $EndComp
 $Comp
-L GND #PWR?
+L GND #PWR07
 U 1 1 56437CAD
 P 4300 4000
-F 0 "#PWR?" H 4300 4000 30  0001 C CNN
+F 0 "#PWR07" H 4300 4000 30  0001 C CNN
 F 1 "GND" H 4300 3930 30  0001 C CNN
 F 2 "" H 4300 4000 60  0001 C CNN
@@
 Connection ~ 3550 3950
 Wire Wire Line
-	1850 2750 2800 2750
-Wire Wire Line
-	2800 2750 2800 4250
-Wire Wire Line
 	2800 4250 3550 4250
 Wire Wire Line
-	1850 2850 2700 2850
-Wire Wire Line
-	2700 2850 2700 4350
-Wire Wire Line
 	2700 4350 3550 4350
 Wire Wire Line
-	1850 2950 2600 2950
-Wire Wire Line
-	2600 2950 2600 4450
-Wire Wire Line
 	2600 4450 3550 4450
 $Comp
-L GND #PWR?
+L GND #PWR08
 U 1 1 56437EE9
 P 4250 4700
-F 0 "#PWR?" H 4250 4700 30  0001 C CNN
+F 0 "#PWR08" H 4250 4700 30  0001 C CNN
 F 1 "GND" H 4250 4630 30  0001 C CNN
 F 2 "" H 4250 4700 60  0001 C CNN
@@
 	4250 4700 4250 4450
 $Comp
-L R_PACK4 RP?
+L R_PACK4 RP1
 U 1 1 56437FB3
-P 2950 3450
-F 0 "RP?" H 2950 3900 40  0000 C CNN
-F 1 "R_PACK4" H 2950 3400 40  0000 C CNN
-F 2 "4X0603" H 2950 3450 60  0001 C CNN
-F 3 "" H 2950 3450 60  0000 C CNN
-	1    2950 3450
-	0    1    -1   0
-$EndComp
-$Comp
-L 3V3 #PWR?
+P 3350 3450
+F 0 "RP1" H 3350 3900 40  0000 C CNN
+F 1 "2k2" H 3350 3400 40  0000 C CNN
+F 2 "kicad-libraries:4X0603" H 3350 3450 60  0001 C CNN
+F 3 "" H 3350 3450 60  0000 C CNN
+	1    3350 3450
+	0    -1   -1   0
+$EndComp
+$Comp
+L 3V3 #PWR09
 U 1 1 56438177
 P 3150 3200
-F 0 "#PWR?" H 3150 3300 40  0001 C CNN
+F 0 "#PWR09" H 3150 3300 40  0001 C CNN
 F 1 "3V3" H 3150 3325 40  0000 C CNN
 F 2 "" H 3150 3200 60  0000 C CNN
@@
 NoConn ~ 3300 3650
 $Comp
-L CRYSTAL X?
-U 1 1 5643858B
-P 5200 4200
-F 0 "X?" H 5200 4350 60  0000 C CNN
-F 1 "CRYSTAL" H 5200 4050 60  0000 C CNN
-F 2 "" H 5200 4200 60  0000 C CNN
-F 3 "" H 5200 4200 60  0000 C CNN
-	1    5200 4200
-	0    1    1    0
-$EndComp
-$Comp
-L 3V3 #PWR?
+L 3V3 #PWR010
 U 1 1 56438992
 P 2000 2350
-F 0 "#PWR?" H 2000 2450 40  0001 C CNN
+F 0 "#PWR010" H 2000 2450 40  0001 C CNN
 F 1 "3V3" H 2000 2475 40  0000 C CNN
 F 2 "" H 2000 2350 60  0000 C CNN
@@
 Wire Wire Line
 	4800 4250 4250 4250
+Text Notes 4950 4700 0    60   ~ 0
+CL = 6,7,12.5pF
+$Comp
+L BATTERY BT1
+U 1 1 564B5B92
+P 5150 5100
+F 0 "BT1" H 5150 5300 50  0000 C CNN
+F 1 "BATTERY" H 5150 4910 50  0000 C CNN
+F 2 "kicad-libraries:BATTERY_HOLDER_2998" H 5150 5100 60  0001 C CNN
+F 3 "" H 5150 5100 60  0000 C CNN
+	1    5150 5100
+	1    0    0    -1
+$EndComp
+$Comp
+L C C3
+U 1 1 564B5C87
+P 4750 5350
+F 0 "C3" V 4600 5250 50  0000 L CNN
+F 1 "100nF" V 4800 5050 50  0000 L CNN
+F 2 "kicad-libraries:0603E" H 4750 5350 60  0001 C CNN
+F 3 "" H 4750 5350 60  0001 C CNN
+	1    4750 5350
+	1    0    0    -1
+$EndComp
+$Comp
+L GND #PWR011
+U 1 1 564B5D5C
+P 4750 5700
+F 0 "#PWR011" H 4750 5700 30  0001 C CNN
+F 1 "GND" H 4750 5630 30  0001 C CNN
+F 2 "" H 4750 5700 60  0001 C CNN
+F 3 "" H 4750 5700 60  0001 C CNN
+	1    4750 5700
+	1    0    0    -1
+$EndComp
+$Comp
+L GND #PWR012
+U 1 1 564B5DAF
+P 5450 5700
+F 0 "#PWR012" H 5450 5700 30  0001 C CNN
+F 1 "GND" H 5450 5630 30  0001 C CNN
+F 2 "" H 5450 5700 60  0001 C CNN
+F 3 "" H 5450 5700 60  0001 C CNN
+	1    5450 5700
+	1    0    0    -1
+$EndComp
+Wire Wire Line
+	5450 5700 5450 5100
+Wire Wire Line
+	4850 5100 4500 5100
+Wire Wire Line
+	4500 5100 4500 4350
+Wire Wire Line
+	4500 4350 4250 4350
+Wire Wire Line
+	4750 5150 4750 5100
+Connection ~ 4750 5100
+Wire Wire Line
+	4750 5700 4750 5550
+$Comp
+L CRYSTAL_3225 X1
+U 1 1 564B61E1
+P 5200 4200
+F 0 "X1" H 5200 4450 60  0000 C CNN
+F 1 "32.768kHz" H 5450 3950 60  0000 C CNN
+F 2 "kicad-libraries:AB26TRQ" H 5200 4200 60  0001 C CNN
+F 3 "" H 5200 4200 60  0000 C CNN
+	1    5200 4200
+	0    -1   -1   0
+$EndComp
+$Comp
+L GND #PWR013
+U 1 1 564B63DC
+P 5500 4500
+F 0 "#PWR013" H 5500 4500 30  0001 C CNN
+F 1 "GND" H 5500 4430 30  0001 C CNN
+F 2 "" H 5500 4500 60  0001 C CNN
+F 3 "" H 5500 4500 60  0001 C CNN
+	1    5500 4500
+	1    0    0    -1
+$EndComp
+Wire Wire Line
+	5500 4500 5500 4350
+Text Notes 5550 5250 0    60   ~ 0
+Digikey 36-2998-ND
+Text Notes 5550 4150 0    60   ~ 0
+ AB26TRQ-32.768kHz-T
+Wire Wire Line
+	1850 2750 2600 2750
+Wire Wire Line
+	2600 2750 2600 4450
+Wire Wire Line
+	2700 4350 2700 2850
+Wire Wire Line
+	2700 2850 1850 2850
+Wire Wire Line
+	2800 4250 2800 2950
+Wire Wire Line
+	2800 2950 1850 2950
+NoConn ~ 1850 3050
 $EndSCHEMATC
