File: hardware/rtc.sch (KiCad schematic (older format))
At the start: 13 parts, among them P1 CON-SENSOR, U1 M24C64, U2 PCF85263AT, U3 DRILL, U4 DRILL, U5 DRILL, U6 DRILL, X1 32.768kHz

Commit message: change rtc battery footprint
Parts:
- C1, C2, C3: symbol C -> C-RESCUE-rtc
Other:
- note added: "364, LR621, AG1\nor\n321, SR616"
Changed lines of the file:
@@
 EESchema Schematic File Version 2
+LIBS:rtc-rescue
 LIBS:power
 LIBS:device
@@
 LIBS:memory
 LIBS:xilinx
-LIBS:special
 LIBS:microcontrollers
 LIBS:dsp
@@
 LIBS:valves
 LIBS:tinkerforge
+LIBS:Zilog
+LIBS:Xicor
 LIBS:video
 LIBS:ttl_ieee
 LIBS:transf
+LIBS:switches
 LIBS:supertex
 LIBS:stm32
 LIBS:stm8
+LIBS:silabs
 LIBS:sensors
 LIBS:rfcom
@@
 LIBS:references
 LIBS:pspice
+LIBS:Power_Management
 LIBS:powerint
+LIBS:Oscillators
+LIBS:onsemi
 LIBS:nxp_armmcu
+LIBS:nordicsemi
 LIBS:msp430
+LIBS:motor_drivers
+LIBS:microchip_pic32mcu
+LIBS:microchip_pic18mcu
 LIBS:microchip_pic16mcu
 LIBS:microchip_pic12mcu
 LIBS:microchip_pic10mcu
+LIBS:microchip_dspic33dsc
+LIBS:maxim
 LIBS:logo
+LIBS:Lattice
+LIBS:ir
 LIBS:hc11
 LIBS:graphic
 LIBS:gennum
 LIBS:ftdi
+LIBS:ESD_Protection
 LIBS:elec-unifil
+LIBS:diode
 LIBS:dc-dc
 LIBS:cmos_ieee
 LIBS:brooktre
+LIBS:analog_devices
+LIBS:Altera
+LIBS:actel
 LIBS:ac-dc
 LIBS:74xgxx
@@
 Copyright Tinkerforge GmbH 2015.\nThis documentation describes Open Hardware and is licensed under the\nCERN OHL v. 1.1.\nYou may redistribute and modify this documentation under the terms of the\nCERN OHL v.1.1. (http://ohwr.org/cernohl). This documentation is distributed\nWITHOUT ANY EXPRESS OR IMPLIED WARRANTY, INCLUDING OF\nMERCHANTABILITY, SATISFACTORY QUALITY AND FITNESS FOR A\nPARTICULAR PURPOSE. Please see the CERN OHL v.1.1 for applicable\nconditions\n
 $Comp
-L GND #PWR01
+L GND-RESCUE-rtc #PWR01
 U 1 1 4CE29748
 P 4700 2550
@@
 $EndComp
 $Comp
-L C C2
+L C-RESCUE-rtc C2
 U 1 1 4C5FD6ED
 P 4500 2400
@@
 SCL
 $Comp
-L GND #PWR02
+L GND-RESCUE-rtc #PWR02
 U 1 1 4C5FD34E
 P 3350 2900
@@
 $EndComp
 $Comp
-L GND #PWR03
+L GND-RESCUE-rtc #PWR03
 U 1 1 4C5FCF5E
 P 2000 2250
@@
 $EndComp
 $Comp
-L GND #PWR04
+L GND-RESCUE-rtc #PWR04
 U 1 1 4C5FCF4F
 P 1400 3300
@@
 $EndComp
 $Comp
-L C C1
+L C-RESCUE-rtc C1
 U 1 1 56437B41
 P 3900 3950
@@
 $EndComp
 $Comp
-L GND #PWR07
+L GND-RESCUE-rtc #PWR07
 U 1 1 56437CAD
 P 4300 4000
@@
 	2600 4450 3550 4450
 $Comp
-L GND #PWR08
+L GND-RESCUE-rtc #PWR08
 U 1 1 56437EE9
 P 4250 4700
@@
 $EndComp
 $Comp
-L C C3
+L C-RESCUE-rtc C3
 U 1 1 564B5C87
 P 4750 5350
@@
 $EndComp
 $Comp
-L GND #PWR011
+L GND-RESCUE-rtc #PWR011
 U 1 1 564B5D5C
 P 4750 5700
@@
 $EndComp
 $Comp
-L GND #PWR012
+L GND-RESCUE-rtc #PWR012
 U 1 1 564B5DAF
 P 5450 5700
@@
 $EndComp
 $Comp
-L GND #PWR013
+L GND-RESCUE-rtc #PWR013
 U 1 1 564B63DC
 P 5500 4500
@@
 	2800 2950 1850 2950
 NoConn ~ 1850 3050
+Text Notes 5650 5600 0    60   ~ 0
+364, LR621, AG1\nor\n321, SR616
 $EndSCHEMATC

Commit message: Add 3d information (tbc)
Parts:
- C1, C2, C3: footprint kicad-libraries:0603E -> kicad-libraries:C0603E; symbol C-RESCUE-rtc -> C
Changed lines of the file:
@@
 EESchema Schematic File Version 2
-LIBS:rtc-rescue
+LIBS:tinkerforge
 LIBS:power
 LIBS:device
@@
 LIBS:contrib
 LIBS:valves
-LIBS:tinkerforge
 LIBS:Zilog
 LIBS:Xicor
@@
 Copyright Tinkerforge GmbH 2015.\nThis documentation describes Open Hardware and is licensed under the\nCERN OHL v. 1.1.\nYou may redistribute and modify this documentation under the terms of the\nCERN OHL v.1.1. (http://ohwr.org/cernohl). This documentation is distributed\nWITHOUT ANY EXPRESS OR IMPLIED WARRANTY, INCLUDING OF\nMERCHANTABILITY, SATISFACTORY QUALITY AND FITNESS FOR A\nPARTICULAR PURPOSE. Please see the CERN OHL v.1.1 for applicable\nconditions\n
 $Comp
-L GND-RESCUE-rtc #PWR01
+L GND #PWR01
 U 1 1 4CE29748
 P 4700 2550
@@
 $EndComp
 $Comp
-L C-RESCUE-rtc C2
+L C C2
 U 1 1 4C5FD6ED
 P 4500 2400
 F 0 "C2" V 4650 2400 50  0000 L CNN
 F 1 "100nF" V 4350 2400 50  0000 L CNN
-F 2 "kicad-libraries:0603E" H 4500 2400 60  0001 C CNN
+F 2 "kicad-libraries:C0603E" H 4500 2400 60  0001 C CNN
 F 3 "" H 4500 2400 60  0001 C CNN
 	1    4500 2400
@@
 SCL
 $Comp
-L GND-RESCUE-rtc #PWR02
+L GND #PWR02
 U 1 1 4C5FD34E
 P 3350 2900
@@
 $EndComp
 $Comp
-L GND-RESCUE-rtc #PWR03
+L GND #PWR03
 U 1 1 4C5FCF5E
 P 2000 2250
@@
 $EndComp
 $Comp
-L GND-RESCUE-rtc #PWR04
+L GND #PWR04
 U 1 1 4C5FCF4F
 P 1400 3300
@@
 $EndComp
 $Comp
-L C-RESCUE-rtc C1
+L C C1
 U 1 1 56437B41
 P 3900 3950
 F 0 "C1" V 4050 3950 50  0000 L CNN
 F 1 "100nF" V 3850 3650 50  0000 L CNN
-F 2 "kicad-libraries:0603E" H 3900 3950 60  0001 C CNN
+F 2 "kicad-libraries:C0603E" H 3900 3950 60  0001 C CNN
 F 3 "" H 3900 3950 60  0001 C CNN
 	1    3900 3950
@@
 $EndComp
 $Comp
-L GND-RESCUE-rtc #PWR07
+L GND #PWR07
 U 1 1 56437CAD
 P 4300 4000
@@
 	2600 4450 3550 4450
 $Comp
-L GND-RESCUE-rtc #PWR08
+L GND #PWR08
 U 1 1 56437EE9
 P 4250 4700
@@
 $EndComp
 $Comp
-L C-RESCUE-rtc C3
+L C C3
 U 1 1 564B5C87
 P 4750 5350
 F 0 "C3" V 4600 5250 50  0000 L CNN
 F 1 "100nF" V 4800 5050 50  0000 L CNN
-F 2 "kicad-libraries:0603E" H 4750 5350 60  0001 C CNN
+F 2 "kicad-libraries:C0603E" H 4750 5350 60  0001 C CNN
 F 3 "" H 4750 5350 60  0001 C CNN
 	1    4750 5350
@@
 $EndComp
 $Comp
-L GND-RESCUE-rtc #PWR011
+L GND #PWR011
 U 1 1 564B5D5C
 P 4750 5700
@@
 $EndComp
 $Comp
-L GND-RESCUE-rtc #PWR012
+L GND #PWR012
 U 1 1 564B5DAF
 P 5450 5700
@@
 $EndComp
 $Comp
-L GND-RESCUE-rtc #PWR013
+L GND #PWR013
 U 1 1 564B63DC
 P 5500 4500
